File: rj45_injector.kicad_pcb (KiCad board)
At the start: 2 copper layers, 45 x 24 mm, 12 parts, among them J1 RJ45_LEDS, J2 RJ45_LEDS, P1 CONN_2, P2 CONN_9, P3 CONN_2, P4 CONN_2, P5 CONN_9, P6 CONN_2

Commit message: updated RJ45 connector modules
Other:
- board text added: "RJ45 INJECTOR V1.1"
- board text removed: "RJ45 INJECTOR V1.0"
